File: FPL/FPL.kicad_pcb (KiCad board)
At the start: 4 copper layers, 100 x 99.8 mm, 62 parts, among them J1 DM3CS-SF, J10 PINHD_1x2_Male, J18 PINHD_1x5_Male, J19 PINHD_1x5_Male, J2 CX90BW1-24P1, J20 PINHD_1x5_Male, J21 PINHD_1x5_Male, J22 PINHD_1x5_Male, J3 PINHD_1x6_Male, J4 2041411-1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

Commit message: code
Routing:
- net PT47A: track 217.2 -> 328.4 mm
- net PT56A: track 180.7 -> 219.8 mm
- net 3V3: track 297.2 -> 302.6 mm
- net GND: track 620.9 -> 616.3 mm, vias 17 -> 16
- net 1V8: track 186.0 -> 184.4 mm
- net Net-(U1H-TMS): track 36.2 -> 34.7 mm
- net Net-(U1A-PT4A): track 7.71 -> 9.03 mm
- net Net-(J2-CC2): track 2.30 -> 3.46 mm
- net LED1: track 7.01 -> 8.10 mm
- net CFG_1: track 11.6 -> 12.5 mm
- net 1V2: track 94.2 -> 95.1 mm
- net MISO: track 25.5 -> 26.3 mm
- net Net-(U5-VDD): track 8.81 -> 9.52 mm
- net Net-(U2-XTAL1/CLKIN): track 18.6 -> 19.1 mm
